File: DACBoard/DACBoard.kicad_pcb (KiCad board)
At the start: 2 copper layers, 80 parts, among them J1 Conn_01x02_Male, J2 Conn_02x20_Odd_Even, J3 Conn_01x02_Male, J4 Conn_01x02_Male, J5 Conn_01x02_Male, J6 Conn_01x04_Male, J7 Conn_01x04_Male, U1 MCP6004

Commit message: Finished first version of design.
Parts:
- moved J3 159.3 mm to (54.4, 73.9), turned to 180 degrees
- moved J1 152.6 mm to (50.0, 75.6), turned to 90 degrees
- moved R35 132.8 mm to (46.5, 70.6)
- moved J5 130.1 mm to (74.0, 79.5), turned to 180 degrees
- moved R71 125.1 mm to (70.6, 86.4), turned to 90 degrees
- moved R54 125.0 mm to (58.8, 56.0)
- moved J4 122.0 mm to (70.5, 58.7)
- moved R18 120.1 mm to (41.0, 79.8)
- moved R62 120.1 mm to (86.4, 52.3), turned to 180 degrees
- moved R72 118.4 mm to (74.2, 93.2), turned to 90 degrees
- moved R36 114.7 mm to (55.5, 87.5), turned to 90 degrees
- moved J7 112.2 mm to (40.6, 75.4)
- moved R67 110.8 mm to (91.4, 61.5)
- moved R53 110.2 mm to (70.6, 63.0), turned to 270 degrees
- moved R60 106.4 mm to (86.4, 58.4), turned to 180 degrees
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Connections:
- J2 pad 29: /+3.3V -> (no net)
- J2 pad 37: /IO_A32 -> (no net)
- J2 pad 38: /IO_A33 -> (no net)
- J2 pad 39: /IO_A34 -> (no net)
- J2 pad 40: /IO_A35 -> (no net)
- R10 pad 2: /IO_A1 -> /IO_A2
- R11 pad 2: /IO_A2 -> /IO_A4
- R12 pad 2: /IO_A3 -> /IO_A6
- R13 pad 2: /IO_A4 -> /IO_A8
- R14 pad 2: /IO_A5 -> /IO_A10
- R15 pad 2: /IO_A6 -> /IO_A12
- R16 pad 2: /IO_A7 -> /IO_A14
- R27 pad 2: /IO_A8 -> /IO_A1
- R28 pad 2: /IO_A9 -> /IO_A3
- R29 pad 2: /IO_A10 -> /IO_A5
- R30 pad 2: /IO_A11 -> /IO_A7
- R31 pad 2: /IO_A12 -> /IO_A9
- R32 pad 2: /IO_A13 -> /IO_A11
- R33 pad 2: /IO_A14 -> /IO_A13
- R46 pad 2: /IO_A17 -> /IO_A18
- R47 pad 2: /IO_A18 -> /IO_A20
- R48 pad 2: /IO_A19 -> /IO_A22
- R49 pad 2: /IO_A20 -> /IO_A24
- R50 pad 2: /IO_A21 -> /IO_A26
- R51 pad 2: /IO_A22 -> /IO_A28
- R52 pad 2: /IO_A23 -> /IO_A30
- R63 pad 2: /IO_A24 -> /IO_A17
- R64 pad 2: /IO_A25 -> /IO_A19
- R65 pad 2: /IO_A26 -> /IO_A21
- R66 pad 2: /IO_A27 -> /IO_A23
- R67 pad 2: /IO_A28 -> /IO_A25
- R68 pad 2: /IO_A29 -> /IO_A27
- R69 pad 2: /IO_A30 -> /IO_A29
Routing:
- net Net-(R25-Pad1): track 149.8 -> 15.5 mm
- net Net-(R23-Pad1): track 141.1 -> 14.3 mm
- net Net-(R16-Pad1): track 3.56 -> 120.0 mm
- net Net-(R21-Pad1): track 123.2 -> 14.3 mm
- net /+5V: track 0.00 -> 104.5 mm
- net Net-(R15-Pad1): track 111.5 -> 12.9 mm
- net Net-(R44-Pad1): track 0.00 -> 93.3 mm
- net Net-(R13-Pad1): track 99.2 -> 14.2 mm
- net Net-(R10-Pad1): track 77.7 -> 14.2 mm
- net Net-(R26-Pad1): track 3.81 -> 63.5 mm
- net Net-(R62-Pad1): track 0.00 -> 53.5 mm
- net Net-(R12-Pad1): track 67.3 -> 14.2 mm
- net Net-(J7-Pad3): track 0.00 -> 51.7 mm
- net Net-(J7-Pad4): track 0.00 -> 48.4 mm
- net Net-(J7-Pad1): track 0.00 -> 25.3 mm
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- added copper zone on B.Cu, net GND
Other:
- board outline added: 104.4 x 69.5 mm
- rule via_min_size: 0.4 -> 0.8
- board text added: "DACBoard for Altera DE1 v0.0.1"
